File: Controller/Controller.kicad_sch (KiCad schematic)
At the start: 24 parts, among them J101 USB_C_Receptacle, J102 Screw_Terminal_01x02, P101 ESProg_Mating_Header, Q101 BSC0503NSI, SW101 RESET, U101 ESP32-S2-WROVER

Commit message: V1.3
Parts:
- added C103, C104, C105: 1uF, Capacitor_SMD:C_0603_1608Metric, symbol Device:C
- added D102, D104: ESDA25P35, Diode_SMD:D_0603_1608Metric, symbol Device:D_Zener
- added D103: ESDA25W, Package_TO_SOT_SMD:SOT-23, symbol Device:D_TVS_x2_AAC
- added R109, R110, R111: 10K, Resistor_SMD:R_0603_1608Metric, symbol Device:R
- added R112: 100K, Resistor_SMD:R_0603_1608Metric, symbol Device:R
- added R113, R114: 1K, Resistor_SMD:R_0603_1608Metric, symbol Device:R
- added SW102: SW_EXT, Connector_PinHeader_2.54mm:PinHeader_1x02_P2.54mm_Vertical, symbol Switch:SW_SPST
- added SW103: SETUP, Button_Switch_SMD:SW_SPST_B3U-1000P, symbol Switch:SW_Push
- added U102: STUSB4500LQTR, Package_DFN_QFN:QFN-24-1EP_4x4mm_P0.5mm_EP2.7x2.7mm, symbol Interface_USB:STUSB4500QTR
Connections:
- net VSNK is gone; now on net VBUS: J102.2 (Pin_2)
- net +3V3: now also R110.2, R111.2, SW102.2 (B)
- net CC1: now also D103.1 (A1), U102.1 (CC1DB), U102.2 (CC1)
- net CC2: now also D103.2 (A2), U102.4 (CC2), U102.5 (CC2DB)
- net GND: now also C103.2, C104.2, C105.2, D102.2 (A), D103.3 (common), D104.2 (A), R109.1, R112.1, SW103.2, U102.10 (GND), U102.12 (ADDR0), U102.13 (ADDR1), U102.22 (VSYS), U102.25 (GND)
- net POK2: now also U102.20 (POWER_OK2)
- net POK3: now also U102.14 (POWER_OK3)
- net SCL: now also U102.7 (SCL)
- net SDA: now also U102.8 (SDA)
- net VBUS: now also C103.1, D104.1 (K), R113.2, R114.1, U102.24 (VDD)
- net VBUS_EN_SNK: now also U102.16 (VBUS_EN_SNK)
- net SW_EXT: now reaches U101.15 (IO12)
- net SW_EXT: now also R109.2, SW102.1 (A)
- net IO18: now reaches U101.21 (IO18)
- net IO18: now also R110.1
- net GP_SETUP: now reaches U101.36 (IO42)
- net GP_SETUP: now also R111.1, SW103.1
- net USB-C PD/GPIO: no longer names the net of D101.1 (K)
- net USB-C PD/GPIO: now also U102.15 (GPIO)
- net USB_VIN: no longer names the net of F101.2, J101.A4 (VBUS), J101.A9 (VBUS), J101.B4 (VBUS), J101.B9 (VBUS)
- net USB_VIN: now also D102.1 (K)
- new net: R113.1, U102.18 (VBUS_VS_DISCH)
- new net: C105.1, U102.23 (VREG_2V7)
- new net: C104.1, U102.21 (VREG_1V2)
- new net: R114.2, U102.9 (DISCH)
- new net RST: R112.2, U102.6 (RESET)
Other:
- removed sheet USB-C PD
- note added: "External switch"
- note added: "Setup button"
- moved on the sheet: D101, J102, Q101, R101, R108
